Commit message: Update robot.urdf

File: src/robot_description/urdf/robot.urdf (robot description, URDF)
Before this commit: robot simple_robot, 1 links, 0 joints
Links:
- added link laser
Joints:
- added joint base_to_laser: type fixed, parent base_link, child laser, origin xyz=0 0 0.2 rpy=0 0 0

Commit message: Update robot.urdf

File: src/robot_description/urdf/robot.urdf (robot description, URDF)
Before this commit: robot simple_robot, 2 links, 1 joints
Links:
- added link base_footprint
Joints:
- added joint footprint_to_base: type fixed, parent base_footprint, child base_link, origin xyz=0 0 0 rpy=0 0 0

Commit message: Update robot.urdf

File: src/robot_description/urdf/robot.urdf (robot description, URDF)
Before this commit: robot simple_robot, 3 links, 2 joints
Links:
- removed link base_footprint
- removed link laser
- added link imu_link; visual box size=0.02 0.02 0.02
- link base_link: geometry visual cylinder length=0.12 radius=0.10
Joints:
- removed joint base_to_laser
- removed joint footprint_to_base
- added joint imu_joint: type fixed, parent base_link, child imu_link, origin xyz=0.0 0.0 0.03 rpy=0.0 0.0 0.0
