Commit message: desc

File: src/robot_description/urdf/recyclebot.urdf (robot description, URDF)
Before this commit: robot recyclebot, 3 links, 2 joints
Links:
- removed link laser
- added link laser_link; visual cylinder length=0.02 radius=0.02
Joints:
- joint laser_joint: child laser -> laser_link

Commit message: Update recyclebot.urdf

File: src/robot_description/urdf/recyclebot.urdf (robot description, URDF)
Before this commit: robot recyclebot, 3 links, 2 joints
Links:
- added link camera_link; visual box size=0.05 0.05 0.05
Joints:
- added joint camera_joint: type fixed, parent base_link, child camera_link, origin xyz=0.0 0.0 0.15 rpy=0 0 0

Commit message: imu link

File: src/robot_description/urdf/recyclebot.urdf (robot description, URDF)
Before this commit: robot recyclebot, 4 links, 3 joints
Links:
- added link imu_link; visual cylinder length=0.05 radius=0.02
Joints:
- added joint imu_joint: type fixed, parent base_link, child imu_link, origin xyz=0.0 0.0 0.1 rpy=0 0 0

Commit message: imu urdf

File: src/robot_description/urdf/recyclebot.urdf (robot description, URDF)
Before this commit: robot recyclebot, 5 links, 4 joints
Joints:
- joint imu_joint: origin xyz=0.0 0.0 0.1 rpy=0 0 0 -> xyz=0.0 0.0 0.1 rpy=0 0 1.5708

Commit message: imu urdf

File: src/robot_description/urdf/recyclebot.urdf (robot description, URDF)
Before this commit: robot recyclebot, 5 links, 4 joints
Joints:
- joint imu_joint: origin xyz=0.0 0.0 0.1 rpy=0 0 1.5708 -> xyz=0.0 0.0 0.1 rpy=0 0 0
